File: kicad/kidNiki/kidNiki.sch (KiCad schematic (older format))
At the start: 134 parts, among them U1 1M, U1 74HC04, U2 2L

Commit message: CourierSud's modifications to the initial Kid Niki schems part 2.
Parts:
- removed D3, D4, D5: IS1588, ~, symbol DIODE
- removed TR7: -, TO92, symbol 2SC1815
- removed VR1: 50k, ~, symbol R
- added D3, D4, D5: 1S1588, symbol D
- added I_BD0, I_CH0, I_OH0, I_OKI0, I_SD0, I_SINH0, I_SOUND0, I_SOUNDIC0, O_AUDIO0: 0, symbol CONN_01X01
- added I_V0, I_V5: 5, symbol CONN_01X01
- added Q7: 2SC945{ECB}, TO92, symbol Q_NPN_ECB
- added RV1: 50k, symbol POT
- C28, C33, C41, C44, C47: value 1uF -> 1u; symbol C -> C-RESCUE-kidNiki
- C31: value 0.47F -> 0.47u; symbol C -> C-RESCUE-kidNiki
- C32, C49: value 0.0033F -> 0.0033u; symbol C -> C-RESCUE-kidNiki
- C34, C35, C38, C39, C63: value 0.001F -> 0.001u; symbol C -> C-RESCUE-kidNiki
- C36: value 0.0065F -> 0.0065u; symbol C -> C-RESCUE-kidNiki
- C37, C45, C50, C51, C60, C61, C70: value 0.022F -> 0.022u; symbol C -> C-RESCUE-kidNiki
- C40: value 12pF -> 12p; symbol C -> C-RESCUE-kidNiki
- C42, C43: value 0.0012F -> 0.0012u; symbol C -> C-RESCUE-kidNiki
- C48: value 1uF -> 0.47u; symbol C -> C-RESCUE-kidNiki
- C52, C53: value 0.027F -> 0.027u; symbol C -> C-RESCUE-kidNiki
- C56, C57, C59, C62: value 0.0068F -> 0.0068u; symbol C -> C-RESCUE-kidNiki
- C58: value 47uF -> 47u; symbol C -> C-RESCUE-kidNiki
- C64, C65, C66, C76: value 0.068F -> 0.068u; symbol C -> C-RESCUE-kidNiki
- C67, C68: value 0.015F -> 0.015u; symbol C -> C-RESCUE-kidNiki
- C69, C73: value 0.01F -> 0.01u; symbol C -> C-RESCUE-kidNiki
- C72, C77: value 0.012F -> 0.012u; symbol C -> C-RESCUE-kidNiki
- Q10: renamed from TR10; value - -> 2SC945{ECB}; symbol 2SC1815 -> Q_NPN_ECB
- Q3: renamed from TR3; value - -> 2SC945{ECB}; symbol 2SC1815 -> Q_NPN_ECB
- Q4: renamed from TR4; value - -> 2SC945{ECB}; symbol 2SC1815 -> Q_NPN_ECB
- Q5: renamed from TR5; value - -> 2SC945{ECB}; symbol 2SC1815 -> Q_NPN_ECB
- Q6: renamed from TR6; value - -> 2SC945{ECB}; symbol 2SC1815 -> Q_NPN_ECB
- Q9: renamed from TR9; value - -> 2SC945{ECB}; symbol 2SC1815 -> Q_NPN_ECB
- R100, R101, R102, R103, R104, R105, R106, R107, R108, R119, R27, R28, R29, R30, R31, R32, R34, R35, R36, R37, R39, R40, R41, R42, R43, R44, R45, R46, R48, R49, R50, R51, R52, R53, R54, R55, R57, R58, R59, R60, R61, R62, R63, R65, R66, R67, R68, R69, R70, R71, R72, R73, R74, R75, R77, R78, R81, R82, R83, R84, R85, R87, R89, R90, R91, R92, R93, R94, R95, R96, R97, R98: symbol R -> R-RESCUE-kidNiki
- R38: value 820k -> 820; symbol R -> R-RESCUE-kidNiki
- R48_2: renamed from R48; symbol R -> R-RESCUE-kidNiki
- R65_1: renamed from R65; symbol R -> R-RESCUE-kidNiki
- R76: value ?k -> 1k; symbol R -> R-RESCUE-kidNiki
- R86: renamed from R66; symbol R -> R-RESCUE-kidNiki
- U1: value 1M -> LM324; symbol LM2902N -> LM324
- U2: value 2L -> LM358; symbol LM2902N -> LM358
- U2: renamed from U?; value 2L -> LM358; symbol LM2902N -> LM358
- renumbered U1 to U3
Connections:
- net labels added: +5V, STV
- wire segments 368 -> 286
Other:
- note added: "R76 is not given in schematics\nFor now, we use 1K until we understand\nthe OKI input signal"
- note added: "There may be issue on the schematics. \nThere is no immediate feedback path \nfrom opamp output to input."
- note added: "This is 820 not 820k"
- note added: "U1 = 1M\nU2 = 2L"
