File: kicad/circus/circus.sch (KiCad schematic (older format))
At the start: 31 parts, among them Q7 2SC1941, U1 74HC04, U8 LM324

Commit message: Added labels to the devices from the schematics and a proper audio out.
Parts:
- added O_AUDIO0: 0, symbol CONN_01X01
- Q7: value 2SC1941 -> 2N4401
- U1, U?: value 74HC04 -> CD4069
- U8: value LM324 -> LM348
Connections:
- net at C6.1: now also O_AUDIO0.1 (P1)
Other:
- note removed: "Audio Out"
Changed lines of the file:
@@
 P 14800 7700
 F 0 "Q7" H 14800 7551 40  0000 R CNN
-F 1 "2SC1941" H 14800 7850 40  0000 R CNN
+F 1 "2N4401" H 14800 7850 40  0000 R CNN
 F 2 "" H 14800 7700 60  0000 C CNN
 F 3 "" H 14800 7700 60  0000 C CNN
@@
 P 18300 1900
 F 0 "U8" H 18350 2100 60  0000 C CNN
-F 1 "LM324" H 18450 1700 50  0000 C CNN
+F 1 "LM348" H 18450 1700 50  0000 C CNN
 F 2 "" H 18300 1900 60  0000 C CNN
 F 3 "" H 18300 1900 60  0000 C CNN
@@
 	1    0    0    1
 $EndComp
-Text Notes 19900 2050 0    60   ~ 0
-Audio Out
 $Comp
 L GND #PWR?
@@
 P 12050 8350
 F 0 "U1" H 12200 8450 40  0000 C CNN
-F 1 "74HC04" H 12250 8250 40  0000 C CNN
+F 1 "CD4069" H 12250 8250 40  0000 C CNN
 F 2 "~" H 12050 8350 60  0000 C CNN
 F 3 "~" H 12050 8350 60  0000 C CNN
@@
 P 9750 8350
 F 0 "U1" H 9900 8450 40  0000 C CNN
-F 1 "74HC04" H 9950 8250 40  0000 C CNN
+F 1 "CD4069" H 9950 8250 40  0000 C CNN
 F 2 "~" H 9750 8350 60  0000 C CNN
 F 3 "~" H 9750 8350 60  0000 C CNN
@@
 P 6750 8350
 F 0 "U1" H 6900 8450 40  0000 C CNN
-F 1 "74HC04" H 6950 8250 40  0000 C CNN
+F 1 "CD4069" H 6950 8250 40  0000 C CNN
 F 2 "~" H 6750 8350 60  0000 C CNN
 F 3 "~" H 6750 8350 60  0000 C CNN
@@
 P 4550 8350
 F 0 "U1" H 4700 8450 40  0000 C CNN
-F 1 "74HC04" H 4750 8250 40  0000 C CNN
+F 1 "CD4069" H 4750 8250 40  0000 C CNN
 F 2 "~" H 4550 8350 60  0000 C CNN
 F 3 "~" H 4550 8350 60  0000 C CNN
@@
 Connection ~ 16950 1800
 Wire Wire Line
-	19900 1900 19600 1900
-Wire Notes Line
-	19850 1850 19850 1950
-Wire Notes Line
-	19850 1950 19950 1950
-Wire Notes Line
-	19950 1950 19950 1850
-Wire Notes Line
-	19950 1850 19850 1850
+	19600 1900 19850 1900
 Wire Wire Line
 	17800 2000 17650 2000
@@
 P 4700 6250
 F 0 "U1" H 4850 6350 40  0000 C CNN
-F 1 "74HC04" H 4900 6150 40  0000 C CNN
+F 1 "CD4069" H 4900 6150 40  0000 C CNN
 F 2 "~" H 4700 6250 60  0000 C CNN
 F 3 "~" H 4700 6250 60  0000 C CNN
@@
 P 6550 6250
 F 0 "U?" H 6700 6350 40  0000 C CNN
-F 1 "74HC04" H 6750 6150 40  0000 C CNN
+F 1 "CD4069" H 6750 6150 40  0000 C CNN
 F 2 "~" H 6550 6250 60  0000 C CNN
 F 3 "~" H 6550 6250 60  0000 C CNN
@@
 	4100 6250 4100 7100
 Connection ~ 5650 7100
+$Comp
+L CONN_01X01 O_AUDIO0
+U 1 1 558D61A1
+P 20050 1900
+F 0 "O_AUDIO0" H 20050 2000 50  0000 C CNN
+F 1 "0" V 20150 1900 50  0000 C CNN
+F 2 "" H 20050 1900 60  0000 C CNN
+F 3 "" H 20050 1900 60  0000 C CNN
+	1    20050 1900
+	1    0    0    -1
+$EndComp
 $EndSCHEMATC

Commit message: Added Rifle Shot and Pipe Hit sounds to Circus schematic.
Parts:
- added C13, C18, C27: 0.05u, ~, symbol C
- added C17, C23: 2.2u, ~, symbol C
- added C19: 0.001u, ~, symbol C
- added C24: 0.022u, ~, symbol C
- added C25, C26: 0.0047u, ~, symbol C
- added D17, D18, D19, D20: DIODE, ~, symbol DIODE
- added I_PIPE_HIT, I_RIFLE_SHOT: 0, symbol CONN_01X01
- added Q1, Q2: ~, symbol 2SC1941
- added Q4, Q5: 2N4093, TO92, symbol BF245A
- added R143, R39, R48: 1000k, ~, symbol R
- added R37, R45, R46: 100k, ~, symbol R
- added R38, R41, R42, R44, R47: 22k, ~, symbol R
- added R40, R49: 100, ~, symbol R
- added R43, R50, R51, R52: 47k, ~, symbol R
- added R53, R54: 10k, ~, symbol R
- added R55: 68k, ~, symbol R
- added U3, U4: ~, ~, symbol 74HC04
- added U5: LM348, symbol LM324
- added U6: MM5837, ~, symbol MM5837
- gave numbers to parts that had none: 1
Connections:
- net +12V: now also R37.1, R39.2, R46.1, R48.1, U6.4 (VCC)
- net GND: now also C17.2, C19.2, C23.1, C25.1, D18.1 (A), D20.1 (A), Q4.3 (D), Q5.2 (S), R143.2, R38.1, R47.2, U3.7 (GND), U3.7 (GND), U4.7 (GND), U4.7 (GND), U6.1 (VDD)
- net VCC: now also U3.14 (VCC), U3.14 (VCC), U4.14 (VCC), U4.14 (VCC)
- net at R13.1, R67.2, U8.13 (-): now also R45.1, R55.1
- new net: C18.2, Q4.1 (G), Q5.1 (G), R143.1
- new net: D20.2 (K), Q5.3 (D), R51.1, U5.12 (+)
- new net: Q2.3 (B), R46.2, R47.1
- new net: Q1.3 (B), R37.2, R38.2
- new net: I_RIFLE_SHOT.1 (P1), Q2.1 (E)
- new net: C27.2, Q2.2 (C), R48.2, U4.1
- new net: I_PIPE_HIT.1 (P1), Q1.1 (E)
- new net: C13.1, Q1.2 (C), R39.1, U3.13
- new net: C13.2, U3.10
- new net: D19.1 (A), U4.2, U4.3
- new net: D17.1 (A), U3.11, U3.12
- new net: C27.1, U4.4
- new net: D19.2 (K), R49.2
- new net: D17.2 (K), R40.2
- new net: C24.2, R53.1, R54.2
- new net: R52.1, R53.2, U5.14
- new net: C23.2, R49.1, R50.2, R51.2
- new net: C17.1, R40.1, R41.2, R42.2
- new net: R41.1, R44.2, U5.2 (-)
- new net: R50.1, R52.2, U5.13 (-)
- new net: C25.2, R54.1, U5.10 (+)
- new net: C24.1, C26.2, U5.8, U5.9 (-)
- new net: D18.2 (K), Q4.2 (S), R42.1, U5.3 (+)
- new net: R43.2, R44.1, U5.1
- new net: C26.1, R55.2
- new net: C18.1, U6.3 (OUT)
- new net: C19.1, R43.1, R45.2
- new net -12V: U6.2 (VGG)
Other:
- note added: "Illegible \nresistance"
- note added: "Mirrored?\n"
- moved on the sheet: C1, C2, C3, C4, C5, D1, D2, D3, D4, D6, I_DUCK_1, Q7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

Commit message: Finsihed Duck 2 and Duck 3 sounds.
Parts:
- added C10, C12, C14: 0.1u, ~, symbol C
- added C11: 0.047u, ~, symbol C
- added C15, C8: 470u, ~, symbol C
- added C9: 0.0047u, ~, symbol C
- added D10, D11, D12, D13, D14, D15, D16, D7, D8, D9: DIODE, ~, symbol DIODE
- added I_DUCK_2, I_DUCK_3: 0, symbol CONN_01X01
- added Q6, Q8: ~, symbol 2SC1941
- added R14, R15, R18, R29: 2200k, ~, symbol R
- added R16, R26, R30, R34: 100k, ~, symbol R
- added R17, R31: 470k, ~, symbol R
- added R19, R23, R24: 3900k, ~, symbol R
- added R20, R21, R22, R25, R28, R32: 1000k, ~, symbol R
- added R27, R36: 47k, ~, symbol R
- added R33, R35: 10k, ~, symbol R
- added U2: ~, ~, symbol 74HC04
- added unit 4 of U3
- added unit 3 of U3
- added unit 2 of U3
- added unit 1 of U3
- Q7: value 2N4401 -> ~
- U1: value CD4069 -> ~
Connections:
- net +12V: now also R25.2, R26.1, R34.1
- net GND: now also C12.1, Q6.1 (E), Q8.1 (E), R33.2, R35.2, U2.7 (GND), U2.7 (GND), U2.7 (GND), U2.7 (GND), U2.7 (GND), U2.7 (GND), U3.7 (GND), U3.7 (GND), U3.7 (GND), U3.7 (GND)
- net VCC: now also U2.14 (VCC), U2.14 (VCC), U2.14 (VCC), U2.14 (VCC), U2.14 (VCC), U2.14 (VCC), U3.14 (VCC), U3.14 (VCC), U3.14 (VCC), U3.14 (VCC)
- net at R13.1, R45.1, R55.1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: now also R27.1, R36.1
- new net: D12.1 (A), D7.1 (A), R26.2
- new net: D7.2 (K), I_DUCK_2.1 (P1)
- new net: D12.2 (K), Q8.3 (B), R35.1
- new net: Q8.2 (C), R17.1, R27.2
- new net: C8.1, R17.2, U2.6
- new net: D13.1 (A), D16.1 (A), R34.2
- new net: D13.2 (K), I_DUCK_3.1 (P1)
- new net: D16.2 (K), Q6.3 (B), R33.1
- new net: Q6.2 (C), R31.1, R36.2
- new net: C15.1, R31.2, U3.2
- new net: C12.2, D11.1 (A), R23.1, R24.2, R25.1
- new net: C11.1, D11.2 (K), D9.2 (K), U2.8
- new net: C11.2, D8.1 (A), R19.2, U2.11
- new net: D8.2 (K), R18.2
- new net: R18.1, R19.1, U2.10, U2.9
- new net: D9.1 (A), R16.2
- new net: C8.2, R14.2, R16.1, R20.2, U2.3
- new net: D10.1 (A), R20.1, R21.1, R24.1
- new net: D10.2 (K), R14.1, U2.4, U2.5
- new net: C10.2, R21.2, R22.1
- new net: D15.1 (A), R22.2, R23.2, R32.1
- new net: C10.1, C9.2, U2.12
- new net: R15.1, U2.13, U2.2
- new net: C9.1, R15.2, U2.1
- new net: C14.1, D14.2 (K), U3.6
- new net: C14.2, R28.2, U3.9
- new net: R28.1, U3.5, U3.8
- new net: D14.1 (A), R30.2
- new net: C15.2, R29.2, R30.1, R32.2, U3.3
- new net: D15.2 (K), R29.1, U3.1, U3.4
Other:
- note added: "pF instead of uF?"
- moved on the sheet: I_DUCK_1, R13, R45, R55

Commit message: The bear sound is now half-complete.
Parts:
- added C40: 0.1u, ~, symbol C
- added C46: 6.8u, ~, symbol C
- added D27, D29, D30, D31: DIODE, ~, symbol DIODE
- added I_BEAR: 0, symbol CONN_01X01
- added Q11, Q12, Q18: ~, symbol 2SC1941
- added R102, R103, R82, R85: 10k, ~, symbol R
- added R104: 100k, ~, symbol R
- added R145, R95: 1000k, ~, symbol R
- added R84: 470k, ~, symbol R
- added R86: 1k, ~, symbol R
- added R87: 5.1k, ~, symbol R
- added R88: 82k, ~, symbol R
- added U12: ~, ~, symbol 74HC04
- added U9: LM348, symbol LM324
Connections:
- net +12V: now also R102.1, R104.1
- net -12V: now also R145.2, R85.2
- net GND: now also C46.1, Q18.1 (E), R103.2, R86.2, U12.7 (GND), U12.7 (GND), U9.3 (+)
- net VCC: now also U12.14 (VCC), U12.14 (VCC)
- new net: D31.2 (K), I_BEAR.1 (P1)
- new net: D30.1 (A), D31.1 (A), R104.2
- new net: D30.2 (K), Q18.3 (B), R103.1
- new net: D29.1 (A), Q18.2 (C), R102.2
- new net: C46.2, D29.2 (K), R145.1, R88.2
- new net: Q11.1 (E), Q12.1 (E), R85.1, R86.1, R87.2
- new net: D27.1 (A), Q11.3 (B), Q12.2 (C), Q12.3 (B), R88.1
- new net: C40.2, D27.2 (K), Q11.2 (C), U9.2 (-)
- new net: R87.1, R95.2, U12.6
- new net: C40.1, R82.2, R84.2, U9.1
- new net: R84.1, R95.1, U12.3
- new net: U12.4, U12.5

Commit message: The Bear sound is complete.
Parts:
- added C39, C41, C45: 0.1u, ~, symbol C
- added C44: 0.0047u, ~, symbol C
- added D28: DIODE, ~, symbol DIODE
- added Q10, Q9: ~, symbol 2SC1941
- added R100, R94: 1000k, ~, symbol R
- added R101, R92: 470k, ~, symbol R
- added R76: 1k, ~, symbol R
- added R77, R83: 10k, ~, symbol R
- added R89, R90: 47k, ~, symbol R
- added R91: 33k, ~, symbol R
- added R93: 5.1k, ~, symbol R
- added unit 5 of U12
- added unit 4 of U12
- added unit 6 of U12
- added unit 1 of U12
- added unit 2 of U9
Connections:
- net -12V: now also R77.1
- net GND: now also R76.1, U12.7 (GND), U12.7 (GND), U12.7 (GND), U12.7 (GND), U9.5 (+)
- net VCC: now also U12.14 (VCC), U12.14 (VCC), U12.14 (VCC), U12.14 (VCC)
- net at R13.1, R27.1, R36.1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: now also R91.1
- net at C46.2, D29.2 (K), R145.1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: now also R101.2, R89.2
- net at R82.1: now also C39.1, R83.2
- new net: C39.2, R91.2
- new net: C41.1, R83.1, R92.1, U9.7
- new net: C44.2, R100.2, R101.1, U12.11
- new net: D28.1 (A), Q10.2 (C), Q10.3 (B), Q9.3 (B), R89.1, R90.1
- new net: R100.1, U12.10, U12.9
- new net: C44.1, C45.1, U12.8
- new net: C45.2, R90.2
- new net: C41.2, D28.2 (K), U9.6 (-)
- new net: Q10.1 (E), Q9.1 (E), R76.2, R77.2
- new net: Q9.2 (C), R93.1
- new net: R92.2, R94.1, U12.1
- new net: R93.2, R94.2, U12.12
- new net: U12.13, U12.2
