File: kicad/carnival/carnival.sch (KiCad schematic (older format))
At the start: 160 parts, among them Q4 2N4093, Q5 2N4093, U6 MM5837, U8 LM348, U9 LM348

Commit message: Bonus #2 is complete.
Parts:
- added C36: 680u, ~, symbol C
- added C37: 0.05u, ~, symbol C
- added C38: 0.1u, ~, symbol C
- added C7: 2.2u, ~, symbol C
- added D23, D24, D25, D26: DIODE, ~, symbol DIODE
- added I_BONUS_2, I_MUSIC: 0, symbol CONN_01X01
- added Q17: ~, symbol 2SC1941
- added R146: 47k, ~, symbol R
- added R68: 470k, ~, symbol R
- added R69: 10k, ~, symbol R
- added R70: 15k, ~, symbol R
- added R71, R73, R80: 1000k, ~, symbol R
- added R72: 750k, ~, symbol R
- added R74: 4.7k, ~, symbol R
- added R75: 5.1k, ~, symbol R
- added R78, R96: 22k, ~, symbol R
- added R79, R81: 100k, ~, symbol R
- added U11: ~, ~, symbol 74HC04
- added unit 1 of U8
Connections:
- net +12V: now also R68.1, R79.1, R80.1
- net -12V: now also R75.2
- net GND: now also R146.2, R78.2, U11.7 (GND), U11.7 (GND), U11.7 (GND), U11.7 (GND), U11.7 (GND), U11.7 (GND), U8.3 (+)
- net VCC: now also U11.14 (VCC), U11.14 (VCC), U11.14 (VCC), U11.14 (VCC), U11.14 (VCC), U11.14 (VCC)
- net at R13.1, R27.1, R36.1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: now also R81.2, R96.2
- new net: I_BONUS_2.1 (P1), Q17.1 (E)
- new net: Q17.3 (B), R78.1, R79.2
- new net: C37.1, Q17.2 (C), R80.2, U11.11
- new net: C37.2, R74.1, U11.8
- new net: U11.10, U11.9
- new net: D26.2 (K), R74.2, R75.1
- new net: C7.1, D24.2 (K), D26.1 (A), R68.2, U8.2 (-)
- new net: C7.2, D24.1 (A), R69.1, U8.1
- new net: D23.1 (A), R69.2, R70.2
- new net: D23.2 (K), R146.1, R81.1
- new net: C36.2, R70.1, U11.2
- new net: R71.1, U11.1, U11.12
- new net: C36.1, R71.2, R72.2, U11.13
- new net: D25.1 (A), R72.1
- new net: C38.2, D25.2 (K), U11.6
- new net: R73.1, U11.4, U11.5
- new net: C38.1, R73.2, U11.3
- new net: I_MUSIC.1 (P1), R96.1
Other:
- note added: "pF again"

Commit message: The "Ranking" sound is complete.
Parts:
- added C33, C51: 0.05u, ~, symbol C
- added C47: 2.2u, ~, symbol C
- added C52: 0.001u, ~, symbol C
- added D32, D33: DIODE, ~, symbol DIODE
- added I_RANKING: 0, symbol CONN_01X01
- added Q16: 2N4093, TO92, symbol BF245A
- added Q19: ~, symbol 2SC1941
- added R107, R108, R99: 47k, ~, symbol R
- added R113: 100, ~, symbol R
- added R114: 22k, ~, symbol R
- added R115: 100k, ~, symbol R
- added R122: 750k, ~, symbol R
- added R123, R144: 1000k, ~, symbol R
- added R98: 220k, ~, symbol R
- added U13: ~, ~, symbol 74HC04
- added U?: LM348, symbol LM324
Connections:
- net +12V: now also R115.1, R123.1
- net GND: now also C47.1, D32.1 (A), Q16.2 (S), R114.2, R144.2, U13.7 (GND), U13.7 (GND), U13.7 (GND), U13.7 (GND)
- net VCC: now also U13.14 (VCC), U13.14 (VCC), U13.14 (VCC), U13.14 (VCC)
- net at R13.1, R27.1, R36.1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: now also R98.1
- new net: I_RANKING.1 (P1), Q19.1 (E)
- new net: D33.1 (A), U13.4, U13.5
- new net: C33.1, U13.6
- new net: C33.2, Q19.2 (C), R123.2, U13.3
- new net: C51.2, C52.1, U13.12
- new net: R122.1, U13.13, U13.2
- new net: C52.2, R122.2, U13.1
- new net: C51.1, Q16.1 (G), R144.1
- new net: D32.2 (K), Q16.3 (D), R108.2, U?.10 (+)
- new net: R98.2, R99.2, U?.8
- new net: R107.2, R99.1, U?.9 (-)
- new net: C47.2, R107.1, R108.1, R113.2
- new net: D33.2 (K), R113.1
- new net: Q19.3 (B), R114.1, R115.2
Other:
- note added: "Mirrored?"

Commit message: The Bonus #1 sound is complete.
Parts:
- added C28, C30, C33: 0.05u, ~, symbol C
- added C29: 0.1u, ~, symbol C
- added C31: 0.0047u, ~, symbol C
- added C32: 6.8u, ~, symbol C
- added D21, D22: DIODE, ~, symbol DIODE
- added I_BONUS_1: 0, symbol CONN_01X01
- added Q3: ~, symbol 2SC1941
- added R56, R62, R66: 100k, ~, symbol R
- added R57, R65: 22k, ~, symbol R
- added R58, R61: 1000k, ~, symbol R
- added R59: 100, ~, symbol R
- added R60: 150k, ~, symbol R
- added R63: 47k, ~, symbol R
- added R64: 470k, ~, symbol R
- added unit 5 of U4
- added unit 6 of U4
- added unit 4 of U4
- added unit 3 of U4
- added U7: LM555N, symbol LM555N
Connections:
- net +12V: now also C32.2, R56.1, R58.1, R63.1, R64.1, U7.4 (R)
- net GND: now also C30.1, C31.1, R57.2, U4.7 (GND), U4.7 (GND), U4.7 (GND), U4.7 (GND), U7.1 (GND)
- net VCC: now also U4.14 (VCC), U4.14 (VCC), U4.14 (VCC), U4.14 (VCC), U7.8 (VCC)
- net at R13.1, R27.1, R36.1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: now also R66.1
- new net: C31.2, R62.2, U7.2 (TR), U7.6 (THR)
- new net: D22.1 (A), U7.3 (Q)
- new net: C30.2, U7.5 (CV)
- new net: R60.2, R62.1, R63.2, U7.7 (DIS)
- new net: I_BONUS_1.1 (P1), Q3.1 (E)
- new net: Q3.3 (B), R56.2, R57.1
- new net: C28.2, Q3.2 (C), R58.2, U4.13
- new net: C28.1, D21.2 (K), U4.10
- new net: U4.11, U4.12
- new net: D21.1 (A), R59.1
- new net: C32.1, R59.2, R64.2, R65.1
- new net: C29.1, R60.1, U4.8
- new net: R61.1, U4.6, U4.9
- new net: C29.2, R61.2, U4.5
- new net: C33.1, D22.2 (K), R65.2
- new net: C33.2, R66.2

Commit message: Finished the "Clang" audio input.  Carnival should now be complete (modulo the inevitable bugs).
Parts:
- added C48: 2.2u, ~, symbol C
- added C49, C50: 0.022u, ~, symbol C
- added C54: 0.5u, ~, symbol C
- added C57, C58: 0.0047u, ~, symbol C
- added C59, C60: 0.0022u, ~, symbol C
- added C61, C62: 0.0033u, ~, symbol C
- added D34: DIODE, ~, symbol DIODE
- added D35, D36, D37, D38: ZENER, ~, symbol ZENER
- added I_CLANG: 0, symbol CONN_01X01
- added Q13, Q14, Q15: ~, TO126, symbol 2SB631
- added Q20: ~, symbol 2SC1941
- added R105, R106, R109, R110, R111, R128, R129, R134, R142: 10k, ~, symbol R
- added R112, R119, R125, R130, R132, R136, R137, R139: 100k, ~, symbol R
- added R116, R120, R133, R141: 330k, ~, symbol R
- added R117: 470k, ~, symbol R
- added R118, R121: 100, ~, symbol R
- added R124: 22k, ~, symbol R
- added R126: 1000k, ~, symbol R
- added R127: 1k, ~, symbol R
- added R131, R135: 2.2k, ~, symbol R
- added R138: 3.3k, ~, symbol R
- added R140: 33k, ~, symbol R
- added R97: 47k, ~, symbol R
- added U10, U14: LM348, symbol LM324
- added unit 4 of U13
- added unit 5 of U13
- added unit 4 of U9
Connections:
- net +12V: now also C48.2, R106.1, R112.1, R125.1, R126.1
- net -12V: now also R109.2, R110.2
- net GND: now also Q13.3 (B), R111.2, R118.2, R124.2, R127.2, R131.2, R135.2, R138.2, U10.12 (+), U10.3 (+), U10.3 (+), U10.5 (+), U13.7 (GND), U13.7 (GND), U14.10 (+), U14.12 (+), U14.3 (+), U14.5 (+)
- net VCC: now also U13.14 (VCC), U13.14 (VCC)
- net at R13.1, R27.1, R36.1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: now also R97.1
- new net: I_CLANG.1 (P1), Q20.1 (E)
- new net: Q20.3 (B), R124.1, R125.2
- new net: C54.1, Q20.2 (C), R126.2, U13.11
- new net: C54.2, D34.2 (K), U13.8
- new net: U13.10, U13.9
- new net: D34.1 (A), R121.1
- new net: C48.1, Q15.3 (B), R112.2, R121.2
- new net: Q15.1 (E), R106.2
- new net: Q13.1 (E), Q14.1 (E), Q15.2 (C)
- new net: Q14.2 (C), R105.1, R110.1, U9.13 (-)
- new net: Q14.3 (B), R117.2, R118.1, R119.2, R130.2, R140.2
- new net: Q13.2 (C), R109.1, R111.1, U9.12 (+)
- new net: C62.1, R140.1, R141.2, R142.2, U14.14
- new net: C60.1, R130.1, R133.2, R134.2, U14.1
- new net: C49.1, R116.2, R117.1, R128.2, U10.14
- new net: C57.1, R119.1, R120.2, R129.2, U10.1
- new net: R105.2, R97.2, U9.14
- new net: D38.1 (A), R142.1, U14.9 (-)
- new net: D38.2 (K), R136.1, U14.8
- new net: C61.2, R141.1, U14.13 (-)
- new net: C61.1, C62.2, R135.1, R136.2
- new net: D37.1 (A), R134.1, U14.6 (-)
- new net: D37.2 (K), R132.1, U14.7
- new net: C59.2, R133.1, U14.2 (-)
- new net: C59.1, C60.2, R131.1, R132.2
- new net: D35.1 (A), R128.1, U10.2 (-)
- new net: D35.2 (K), R137.1, U10.1
- new net: C50.2, R116.1, U10.13 (-)
- new net: C49.2, C50.1, R127.1, R137.2
- new net: D36.1 (A), R129.1, U10.6 (-)
- new net: D36.2 (K), R139.1, U10.7
- new net: C58.2, R120.1, U10.2 (-)
- new net: C57.2, C58.1, R138.1, R139.2
