File: kicad/tb303/tb303.sch (KiCad schematic (older format))
At the start: 69 parts, among them IC10 4050, IC11 AN6562, IC12 4066, IC9 4174, Q28 2SK30

Commit message: Additional work on the 303 + a new MAME.lib addition.
Parts:
- added C54: 0.047u, ~, symbol C
- added C55: 2.9375u, ~, symbol C
- added C62: 0.0285u, ~, symbol C
- added C72: 0.625u, ~, symbol C
- added D34, D35, D36, D37: DIODE, ~, symbol DIODE
- added IC13: MC14013, MODULE, symbol MC14013
- added O_GATE: 0, symbol CONN_01X01
- added Q35, Q37, Q40, Q41: ~, symbol 2SC1941
- added Q36, Q38: ~, TO126, symbol 2SB631
- added Q39: 2SK30, ~, symbol BF245A
- added R133: 2.2k, ~, symbol R
- added R137: 1k, ~, symbol R
- added R138: 68k, ~, symbol R
- added R139, R140, R141: 100k, ~, symbol R
- added R142, R143, R144, R145, R148: 10k, ~, symbol R
- added R146, R151: 22k, ~, symbol R
- added R147, R150: 22, ~, symbol R
- added R149: 20k, ~, symbol R
- added R152: 100, ~, symbol R
Connections:
- net GND: now also C55.2, C62.2, IC13.10 (R2), IC13.7 (VSS), IC13.8 (S2), Q35.1 (E), Q37.1 (E), Q39.1 (G), Q39.2 (S), R140.2, R144.2, R145.2, R151.2
- net STV: now also C72.1, IC13.14 (VDD), Q40.2 (C), Q41.2 (C), R139.1, R142.1, R147.1, R149.1, R150.1
- net at I_7.1 (P1): now also IC13.9 (D2)
- net at I_8.1 (P1): now also IC9.9 (CLK), R59.2, IC13.11 (C2)
- net at I_9.1 (P1): now also R146.2
- new net: D34.2 (K), O_GATE.1 (P1)
- new net: D34.1 (A), R137.1
- new net: IC13.12 (Q2NOT), R141.1
- new net: D35.1 (A), Q36.2 (C), R137.2, R145.1
- new net: D35.2 (K), R133.2
- new net: Q35.3 (B), R140.1, R141.2
- new net: Q35.2 (C), R139.2
- new net: Q36.1 (E), R147.2
- new net: C72.2, Q36.3 (B), R142.2, R143.1
- new net: C54.2, Q37.2 (C), R143.2
- new net: Q37.3 (B), R144.1, R146.1
- new net: Q38.3 (B), R148.1, R149.2
- new net: C54.1, R148.2
- new net: C55.1, Q38.1 (E), R150.2
- new net: D36.1 (A), D37.1 (A), Q38.2 (C), R151.1
- new net: D37.2 (K), R152.2
- new net: C62.1, Q41.3 (B), R138.2, R152.1
- new net: Q40.3 (B), Q41.1 (E)
- new net: Q39.3 (D), Q40.1 (E)
Other:
- note added: "ACCENT"
- note added: "ENV"
- note added: "J4"
- note added: "VCA"
- note added: "White triangle?"
- moved on the sheet: I_7, I_8, I_9

Commit message: ENV is done now.
Parts:
- added ACCENT: 50k(B), ~, symbol POT
- added D26, D27, D28: DIODE, ~, symbol DIODE
- added ENV.DECAY: 1000k(A), ~, symbol POT
- added ENV.MOD: 50k(A), ~, symbol POT
- added unit 1 of IC12
- added unit 2 of IC12
- added R117: 22k, ~, symbol R
- added R61: 10k, ~, symbol R
Connections:
- net +5V: now also TUNING.3, R117.1
- net GND: now also ACCENT.1, D26.2 (K)
- net at Q35.2 (C), R139.2: now also IC12.13 (ON), IC12.5 (ON)
- net at R138.1: now also ENV.DECAY.1, IC12.3 (O/I)
- net at Q39.3 (D), Q40.1 (E): now also ENV.MOD.3, IC12.1 (I/O)
- new net: ACCENT.3, IC12.2 (O/I)
- new net: D28.1 (A), ENV.DECAY.2, ENV.DECAY.3, IC12.4 (I/O)
- new net: D27.1 (A), D28.2 (K)
- new net: D26.1 (A), D27.2 (K), R117.2
- new net: ENV.MOD.1, R61.1
Other:
- note added: "DECAY"
- note added: "VR5"
- note added: "VR6"
- note added: "VR7"

Commit message: The VCA is now complete as well.
Parts:
- added C21, C22: 0.01u, ~, symbol C
- added C36: 0.033u, ~, symbol C
- added C37, C40: 0.625u, ~, symbol C
- added C38: 0.02u, ~, symbol C
- added C41: 0.1u, ~, symbol C
- added C42: 0.0285u, ~, symbol C
- added D27: DIODE, ~, symbol DIODE
- added IC15: BA662, ~, symbol BA662
- added Q27: ~, TO126, symbol 2SB631
- added Q32: ~, symbol 2SC1941
- added R119, R127: 47k, ~, symbol R
- added R120, R129, R134: 22k, ~, symbol R
- added R121, R128, R131: 220k, ~, symbol R
- added R122: 100k, ~, symbol R
- added R123: 1500k, ~, symbol R
- added R124, R125, R126, R162: 2.2k, ~, symbol R
- added R130, R132: 100, ~, symbol R
- renumbered Q27 to Q31
Connections:
- net +5V: now also R126.2, R162.1
- net GND: now also C36.2, C37.2, C40.2, C41.2, C42.2, IC15.5 (-V), R130.2
- net STV: now also IC15.4 (IN1), IC15.9 (+V), Q27.1 (E), R123.1; no longer Q31.1 (E)
- net at R133.1: now also R131.1
- net at Q25.2 (C): now also Q27.3 (B); no longer Q31.3 (B)
- net at D25.1 (A): now also Q27.2 (C); no longer Q31.2 (C)
- net at D36.2 (K): now also R134.2
- new net: Q31.1 (E), R131.2
- new net: D27.2 (K), IC15.1 (C), Q31.2 (C)
- new net: C42.1, Q31.3 (B), R123.2, R132.1
- new net: IC15.2 (-), R125.1
- new net: IC15.3 (+), R121.2, R122.2, R124.1
- new net: IC15.6 (OUT1), IC15.7 (IN2), R127.2, R128.2
- new net: C38.2, IC15.8 (OUT2)
- new net: C37.1, R124.2, R125.2, R126.1
- new net: C21.2, R121.1
- new net: C22.2, R122.1
- new net: C41.1, Q32.3 (B), R134.1
- new net: Q32.1 (E), R130.1
- new net: Q32.2 (C), R132.2
- new net: R127.1, R129.2
- new net: C40.1, R128.1, R129.1, R162.2
- new net: D27.1 (A), R120.2
- new net: C36.1, R119.2, R120.1
Other:
- note added: "http://wiki.openmusiclabs.com/wiki/x0xb0x"
- moved on the sheet: D36, Q31, R133

Commit message: The TB-303 is complete - with numerous curiosities.
Parts:
- added C13, C14, C15, C17, C22, C23, C29: 0.02u, ~, symbol C
- added C16, C30: 0.625u, ~, symbol C
- added C18: 0.018u, ~, symbol C
- added C19, C24, C26: 0.033u, ~, symbol C
- added C25, C27: 0.1u, ~, symbol C
- added C28: 2.9375u, ~, symbol C
- added CUTOFF_FREQ., RESONANCE1, RESONANCE2: 50k(B), ~, symbol POT
- added Q10, Q9: ~, TO126, symbol 2SB631
- added Q11, Q12A, Q12B, Q13, Q14, Q15, Q16, Q17, Q18, Q19, Q20, Q21A, Q21B, Q22A, Q22B, Q23: ~, symbol 2SC1941
- added R108, R110, R111, R67, R68, R69, R70, R71, R98: 2.2k, ~, symbol R
- added R109, R112, R115, R116, R47, R64, R65, R94, R96, R97: 10k, ~, symbol R
- added R113, R114, R66, R72, R73, R99: 100k, ~, symbol R
- added R46: 47k, ~, symbol R
- added R62, R63: 220k, ~, symbol R
- added R95: 100, ~, symbol R
- added TM3: 470k, ~, symbol POT
- added VOLUME: 50k(A), ~, symbol POT
Connections:
- net +5V: now also R116.1, R65.2, R66.1, R68.2
- net GND: now also C13.2, C16.2, C22.2, C28.2, C29.2, C30.2, Q9.2 (C), R108.2, R109.2, R64.2, R94.1, R96.2, RESONANCE2.1, VOLUME.1
- net STV: now also CUTOFF_FREQ..3, Q18.2 (C), R95.1
- net at S1.2 (PM): now also R62.1
- net at ENV.MOD.2: now also R63.1
- net at R61.2: now also Q10.2 (C), Q11.1 (E), Q9.1 (E), R47.2, R71.2
- net at ACCENT.2: now also R119.1, R46.2
- net at C21.1: now also C14.2, RESONANCE2.3
- net at C22.1: now also C15.2, RESONANCE2.2
- net at C38.1: now also VOLUME.3
- new net: R46.1, RESONANCE1.1
- new net: R72.1, RESONANCE1.2
- new net: C13.1, RESONANCE1.3
- new net: CUTOFF_FREQ..1, R47.1
- new net: CUTOFF_FREQ..2, TM3.3
- new net: C17.1, R62.2
- new net: C17.2, Q12A.3 (B), R70.1
- new net: C16.1, R68.1, R70.2, R98.2
- new net: Q12B.3 (B), R97.2, R98.1
- new net: C23.1, R97.1
- new net: C23.2, Q18.1 (E), R94.2
- new net: Q12A.1 (E), Q12B.1 (E), R69.1
- new net: Q11.2 (C), R69.2
- new net: Q10.1 (E), Q11.3 (B), R73.2
- new net: Q10.3 (B), R63.2, R71.1, R72.2
- new net: Q9.3 (B), R64.1, R65.1
- new net: C18.2, Q12B.2 (C), Q15.1 (E)
- new net: C18.1, Q12A.2 (C), Q13.1 (E)
- new net: R73.1, TM3.1, TM3.2
- new net: Q18.3 (B), R67.2, R99.2
- new net: C22.1, R66.2, R99.1
- new net: C15.1, R67.1
- new net: C19.1, Q13.2 (C), Q13.3 (B), Q14.1 (E)
- new net: C19.2, Q15.2 (C), Q15.3 (B), Q17.1 (E)
- new net: C24.1, Q14.2 (C), Q14.3 (B), Q16.1 (E)
- new net: C24.2, Q17.2 (C), Q17.3 (B), Q23.1 (E)
- new net: C25.1, C26.1, Q16.2 (C), Q16.3 (B), Q22A.1 (E)
- new net: C26.2, C27.1, Q22B.1 (E), Q23.2 (C), Q23.3 (B)
- new net: C28.1, Q19.2 (C), Q22A.2 (C), Q22B.2 (C), R110.1, R111.1, R115.1, R95.2
- new net: C30.1, Q22A.3 (B), Q22B.3 (B), R115.2
- new net: C27.2, Q21A.3 (B), R113.1
- new net: C29.1, R112.1, R113.2, R114.2, R116.2
- new net: Q20.3 (B), R109.1, R112.2
- new net: Q20.1 (E), R108.1
- new net: Q20.2 (C), Q21A.1 (E), Q21B.1 (E)
- new net: Q19.3 (B), Q21B.2 (C), R110.2
- new net: C25.2, Q21B.3 (B), R114.1
- new net: Q21A.2 (C), R111.2
- new net: C14.1, Q19.1 (E), R96.1
Other:
- note added: "2SC2291"
- note added: "CONNECTED TO POWER SUPPLY"
- note added: "DOTTED LINE?"
- note added: "FREQ"
- note added: "HEADPHONE"
- note added: "MIXER"
- note added: "VCF"
- note added: "VR3"
- note added: "VR4"
- note added: "VR8"
- note added: "WIDTH"
- moved on the sheet: C21, C22, C36, C37, C38, C40, C41, C42, D27, D36, ENV.DECAY, IC12A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
