File: kicad/congoBongo/congoBongo.sch (KiCad schematic (older format))
At the start: 23 parts, among them U13 MB3614, U6 7416

Commit message: Finished the Bass Drum, Conga(L), Conga(H), and Rim sounds.
Parts:
- removed unit 2 of U13
- added C26, C32: 0.068u, ~, symbol C
- added C27, C30, C31, C33, C35, C36: 0.033u, ~, symbol C
- added C28, C34: 47u, ~, symbol C
- added C29, C37, C44: 1u, ~, symbol C
- added C38: 0.01u, ~, symbol C
- added C39: 0.0033u, ~, symbol C
- added C40: 2.2u, ~, symbol C
- added C41, C42: 0.0068u, ~, symbol C
- added C43: 0.047u, ~, symbol C
- added D2, D3, D4: DIODE, ~, symbol DIODE
- added R31, R37, R41, R47, R51, R56: 10k, ~, symbol R
- added R32, R33, R34, R35, R42, R43, R44, R47: 47k, ~, symbol R
- added R36, R46, R52, R53, R54, R55: 22k, ~, symbol R
- added R38, R48, R58: 1000k, ~, symbol R
- added R39: 330, ~, symbol R
- added R40, R50: 390k, ~, symbol R
- added R49: 220, ~, symbol R
- added R57: 4.7k, ~, symbol R
- added R59: 470, ~, symbol R
- added R60, R61: 2200k, ~, symbol R
- added R62: 200k, ~, symbol R
- added unit 2 of U6
- added U?: MB3614, symbol LM324
- C20: renamed from C?; value C -> 0.068u
- C21, C25: renamed from C?; value C -> 1u
- C22: renamed from C?; value C -> 47u
- C23, C24: renamed from C?; value C -> 0.1u
- R21, R24, R27: renamed from R?; value R -> 10k
- R22, R23, R25: renamed from R?; value R -> 47k
- R26: renamed from R?; value R -> 22k
- R28: renamed from R?; value R -> 470k
- R29: renamed from R?; value R -> 1k
- R30: renamed from R?; value R -> 240k
- gave numbers to parts that had none: 1
Connections:
- net +12V: now also R31.1, R37.1, R41.1, R47.1, R51.1, R57.1
- net GND: now also C28.2, C34.2, C40.2, C43.2, R32.2, R33.2, R35.2, R39.2, R42.2, R43.2, R47.2, R49.2, R52.2, R53.2, R55.2, R59.2, U6.3, U6.7 (GND)
- net VCC: now also U6.14 (VCC)
- net at I_CONGA_L.1 (P1): now also U6.5
- net at I_CONGA_H.1 (P1): now also U6.13
- net at I_RIM.1 (P1): now also U6.11
- net at U6.6: now also C26.2, R31.2
- net at U6.12: now also C32.2, R41.2
- net at U6.10: now also C38.2, R51.2
- net at R30.1: now also R40.1, R50.1, R62.1
- net at U13.10 (+): now also R34.1, R35.1, R36.2
- net at U13.8: now also C29.2, C31.1, R38.1
- net at U13.9 (-): now also C30.2, R38.2
- net at U13.1: now also C36.1, C37.2, R48.1
- net at U13.2 (-): now also C35.2, R48.2
- net at U13.3 (+): now also R43.1, R44.1, R46.2
- new net: C27.2, D2.1 (A), R33.1
- new net: C26.1, D2.2 (K), R32.1
- new net: C29.1, R40.2
- new net: C30.1, C31.2, R39.1
- new net: C27.1, R34.2
- new net: C28.1, R36.1, R37.2
- new net: C33.2, D3.1 (A), R47.1
- new net: C32.1, D3.2 (K), R42.1
- new net: C37.1, R50.2
- new net: C35.1, C36.2, R49.1
- new net: C33.1, R44.2
- new net: C34.1, R46.1, R47.2
- new net: C39.2, D4.1 (A), R53.1
- new net: C38.1, D4.2 (K), R52.1
- new net: C42.1, C44.2, R58.1, R61.1, U?.1
- new net: C41.2, R58.2, R60.2, U?.2 (-)
- new net: R54.1, R55.1, R56.2, U?.3 (+)
- new net: C44.1, R62.2
- new net: C41.1, C42.2, R59.1
- new net: C39.1, R54.2
- new net: C40.1, R56.1, R57.2
- new net: C43.1, R60.1, R61.2
Other:
- note added: "SJ?"
- moved on the sheet: C20, C21, C22, C23, C24, C25, D1, I_BASS_DRUM, R21, R22, R23, R24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

Commit message: Upper-left corner is nearly complete.
Parts:
- added C45: 33u, ~, symbol C
- added C46: 0.1u, ~, symbol C
- added C47: 470u, ~, symbol C
- added C48: 0.0015u, ~, symbol C
- added C49: 220u, ~, symbol C
- added C50: 0.0039u, ~, symbol C
- added C51: 1u, ~, symbol C
- added D5: DIODE, ~, symbol DIODE
- added R63, R64: 22k, ~, symbol R
- added R65, R66, R67, R68, R69: 20k, ~, symbol R
- added R78: 47k, ~, symbol R
- added U17: MB3614, symbol LM324
- added U18: 4011, symbol 4011
- added U?: 4538, symbol 4538
Connections:
- net labels added: +5V
- wire segments 140 -> 188
Other:
- note added: "Schematic says 4001B (NOR gate) \nbut shows AND gate (4011B)"

Commit message: Fixed 4001 (NOR array) bug + added a bunch more in the lower-left corner.
Parts:
- removed U18: 4011, symbol 4011
- added C52, C53, C55: 1u, ~, symbol C
- added C56: 10u, ~, symbol C
- added D6, D7: DIODE, ~, symbol DIODE
- added I_GORILLA: 0, symbol CONN_01X01
- added R70: 100k, ~, symbol R
- added R71: 150k, ~, symbol R
- added R72: 330k, ~, symbol R
- added R73: 1k, ~, symbol R
- added R76, R81: 10k, ~, symbol R
- added R77, R80: 20k, ~, symbol R
- added R79: 22k, ~, symbol R
- added unit 4 of U17
- added unit 2 of U17
- added U18, U?: 4001, symbol 4001
- added unit 2 of U19
- I_BASS_DRUM, I_CONGA_H, I_CONGA_L, I_RIM: value ~ -> 0
- gave numbers to parts that had none: 1
Connections:
- wire segments 188 -> 256
Other:
- note removed: "Schematic says 4001B (NOR gate) \nbut shows AND gate (4011B)"
- moved on the sheet: C51, R78, U19A

Commit message: Congo Bongo is finished save for 2 unknown chips and uncertainty about our ability to handle 4538Bs.
Parts:
- added C54: 1u, ~, symbol C
- added C57: 0.047u, ~, symbol C
- added C58 (x2), C62: 0.022u, ~, symbol C
- added C59: 10u, ~, symbol C
- added D8: DIODE, ~, symbol DIODE
- added Q2: 2SC1941, symbol 2SC1941
- added R74: 1k, ~, symbol R
- added R75: 470k, ~, symbol R
- added R82, R87, R90: 100k, ~, symbol R
- added R83, R84, R85, R86: 51k, ~, symbol R
- added R88: 2.2k, ~, symbol R
- added R89, R91: 10k, ~, symbol R
- added R92, R93: 15k, ~, symbol R
- added U16: MB3614, symbol LM324
- added unit 1 of U17
Connections:
- net labels added: +6V
- wire segments 256 -> 424
Other:
- note added: "G501534"
- note added: "HM5837"
- moved on the sheet: C56, D7, R81, U6B

Commit message: Define and fill in missing chips.
Parts:
- added O_AUDIO0: 0, symbol CONN_01X01
- added U15: G501534, ~, symbol G501534
- added U20: MM5837, ~, symbol MM5837
Connections:
- wire segments 424 -> 337
Other:
- note removed: "G501534"
- note removed: "HM5837"
- moved on the sheet: C45, C46, C58

Commit message: congoBongo: - Added a power section. - Fixed all issues reported by electrical rules check. - Add a "0" to input pins so that kicad stops complaining about   missing annotation. - Fixed MB5837 symbol. Power pins need to be "Power Input" pins.
Parts:
- added I_V0, I_V12, I_V5, I_V6: 0, symbol CONN_01X01
- C20, C21, C22, C23, C24, C25, C26, C27, C28, C29, C30, C31, C32, C33, C34, C35, C36, C37, C38, C39, C40, C41, C42, C43, C44, C45, C46, C47, C48, C49, C50, C51, C52, C53, C54, C55, C56, C57, C58, C59, C62: symbol C -> C-RESCUE-congoBongo
- C60: renamed from C58; symbol C -> C-RESCUE-congoBongo
- R21, R22, R23, R24, R25, R26, R27, R28, R29, R30, R31, R32, R33, R34, R35, R36, R37, R38, R39, R40, R41, R42, R44, R46, R47, R48, R49, R50, R51, R52, R53, R54, R55, R56, R57, R58, R59, R60, R61, R62, R63, R64, R65, R66, R67, R68, R69, R70, R71, R72, R73, R74, R75, R76, R77, R78, R79, R80, R81, R82, R83, R84, R85, R86, R87, R88, R89, R90, R91, R92, R93: symbol R -> R-RESCUE-congoBongo
- R43: renamed from R47; symbol R -> R-RESCUE-congoBongo
- R45: renamed from R43; symbol R -> R-RESCUE-congoBongo
- gave numbers to parts that had none: 2
- renumbered I_BASS_DRUM to I_BASS_DRUM0, I_CONGA_H to I_CONGA_H0, I_CONGA_L to I_CONGA_L0, I_GORILLA to I_GORILLA0, I_RIM to I_RIM0
Connections:
- net VCC is gone; now on net +6V: U6.14 (VCC), U6.14 (VCC), U6.14 (VCC), U6.14 (VCC), U6.14 (VCC)
- net VDD is gone; now on net +5V: U18.14 (VDD), U18.14 (VDD), U18.14 (VDD), U18.14 (VDD), U19.16 (VDD), U19.16 (VDD)
- net VSS is gone; now on net GND: U18.7 (VSS), U18.7 (VSS), U18.7 (VSS), U18.7 (VSS), U19.8 (VSS), U19.8 (VSS)
- net +12V: now also U13.4 (V+), U16.4 (V+), U17.4 (V+), I_V12.1 (P1)
- net +5V: now also I_V5.1 (P1)
- net +6V: now also I_V6.1 (P1)
- net GND: now also U13.11 (V-), U16.11 (V-), U17.11 (V-), I_V0.1 (P1)
- net at C42.1, C44.2, R58.1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: now also U13.7; no longer U13.1
- net at C41.2, R58.2, R60.2: now also U13.6 (-); no longer U13.2 (-)
- net at R54.1, R55.1, R56.2: now also U13.5 (+); no longer U13.3 (+)
- no-connect marks 0 -> 12
Other:
- moved on the sheet: C45

Commit message: More work on congoBongo.
Parts:
- added C61: 1u, ~, symbol C-RESCUE-congoBongo
- added R94: 51k, ~, symbol R-RESCUE-congoBongo
- added unit 1 of U6
- D1, D2, D3, D5, D6, D8: value DIODE -> 1S2075
- Q2: value 2SC1941 -> 2SC1941{ECB}
Connections:
- net +5V: now also U6.14 (VCC), U6.14 (VCC), U6.14 (VCC), U6.14 (VCC), U6.14 (VCC), U6.14 (VCC)
- net +6V: no longer U6.14 (VCC), U6.14 (VCC), U6.14 (VCC), U6.14 (VCC), U6.14 (VCC)
- net GND: now also U6.1, U6.7 (GND)
- net at O_AUDIO0.1 (P1), R30.1, R40.1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: now also R94.1; no longer U15.3 (P3)
- new net: C61.2, U15.3 (P3)
- new net: C61.1, R94.2
- no-connect marks 12 -> 13
Changed lines of the file:
@@
 P 22750 2950
 F 0 "D1" H 22750 3050 40  0000 C CNN
-F 1 "DIODE" H 22750 2850 40  0000 C CNN
+F 1 "1S2075" H 22750 2850 40  0000 C CNN
 F 2 "~" H 22750 2950 60  0000 C CNN
 F 3 "~" H 22750 2950 60  0000 C CNN
@@
 P 22750 7500
 F 0 "D2" H 22750 7600 40  0000 C CNN
-F 1 "DIODE" H 22750 7400 40  0000 C CNN
+F 1 "1S2075" H 22750 7400 40  0000 C CNN
 F 2 "~" H 22750 7500 60  0000 C CNN
 F 3 "~" H 22750 7500 60  0000 C CNN
@@
 P 22750 12100
 F 0 "D3" H 22750 12200 40  0000 C CNN
-F 1 "DIODE" H 22750 12000 40  0000 C CNN
+F 1 "1S2075" H 22750 12000 40  0000 C CNN
 F 2 "~" H 22750 12100 60  0000 C CNN
 F 3 "~" H 22750 12100 60  0000 C CNN
@@
 P 7200 2100
 F 0 "D5" H 7200 2200 40  0000 C CNN
-F 1 "DIODE" H 7200 2000 40  0000 C CNN
+F 1 "1S2075" H 7200 2000 40  0000 C CNN
 F 2 "~" H 7200 2100 60  0000 C CNN
 F 3 "~" H 7200 2100 60  0000 C CNN
@@
 P 7400 11800
 F 0 "D6" H 7400 11900 40  0000 C CNN
-F 1 "DIODE" H 7400 11700 40  0000 C CNN
+F 1 "1S2075" H 7400 11700 40  0000 C CNN
 F 2 "~" H 7400 11800 60  0000 C CNN
 F 3 "~" H 7400 11800 60  0000 C CNN
@@
 P 11950 21700
 F 0 "D8" H 11950 21800 40  0000 C CNN
-F 1 "DIODE" H 11950 21600 40  0000 C CNN
+F 1 "1S2075" H 11950 21600 40  0000 C CNN
 F 2 "~" H 11950 21700 60  0000 C CNN
 F 3 "~" H 11950 21700 60  0000 C CNN
@@
 P 10050 21700
 F 0 "Q2" H 10050 21551 40  0000 R CNN
-F 1 "2SC1941" H 10050 21850 40  0000 R CNN
+F 1 "2SC1941{ECB}" H 10050 21850 40  0000 R CNN
 F 2 "" H 10050 21700 60  0000 C CNN
 F 3 "" H 10050 21700 60  0000 C CNN
@@
 	28700 3050 30100 3050
 Wire Wire Line
-	30100 2800 30100 20500
+	30100 20500 30100 2800
 Wire Wire Line
 	28700 16900 30100 16900
@@
 	3150 11100 3100 11100
 Wire Wire Line
-	3100 11100 3100 10900
+	3100 11100 3100 10500
 Wire Wire Line
-	3100 10900 4150 10900
+	3100 10500 4150 10500
 Wire Wire Line
 	3150 11300 3000 11300
 Wire Wire Line
-	3000 11300 3000 10850
-Wire Wire Line
-	3000 10850 3550 10850
+	3000 11300 3000 10250
 Wire Wire Line
 	2750 10250 3650 10250
 Wire Wire Line
-	3550 10850 3550 10250
-Wire Wire Line
 	2750 10250 2750 11700
-Connection ~ 3550 10250
 Wire Wire Line
 	3150 11500 2750 11500
 Connection ~ 2750 11500
 Wire Wire Line
-	4150 10900 4150 10000
+	4150 10500 4150 10000
 Wire Wire Line
 	4150 10250 4050 10250
@@
 	6400 19150 6550 19150
 Wire Wire Line
-	30100 20500 23650 20500
+	28650 20500 30100 20500
+Wire Wire Line
+	23650 20500 27350 20500
 Wire Wire Line
 	23350 21100 23350 22450
@@
 Connection ~ 11400 19850
 Wire Wire Line
-	30400 2800 30100 2800
+	30100 2800 30400 2800
 Wire Wire Line
 	3600 2150 3600 2700
@@
 Connection ~ 1150 1050
 Wire Wire Line
-	950  1750 1750 1750
-Wire Wire Line
 	1150 1750 1150 1700
 Wire Wire Line
@@
 Connection ~ 1150 1750
 Wire Wire Line
-	950  2150 1750 2150
-Wire Wire Line
 	1150 2150 1150 2100
 Wire Wire Line
 	1400 2150 1400 2200
 Connection ~ 1150 2150
-$Comp
-L VDD #PWR067
-U 1 1 55A65399
-P 1750 1700
-F 0 "#PWR067" H 1750 1550 50  0001 C CNN
-F 1 "VDD" H 1750 1850 50  0000 C CNN
-F 2 "" H 1750 1700 60  0000 C CNN
-F 3 "" H 1750 1700 60  0000 C CNN
-	1    1750 1700
-	1    0    0    -1
-$EndComp
-$Comp
-L VSS #PWR068
-U 1 1 55A65587
-P 1750 2100
-F 0 "#PWR068" H 1750 1950 50  0001 C CNN
-F 1 "VSS" H 1750 2250 50  0000 C CNN
-F 2 "" H 1750 2100 60  0000 C CNN
-F 3 "" H 1750 2100 60  0000 C CNN
-	1    1750 2100
-	1    0    0    -1
-$EndComp
-Wire Wire Line
-	1750 1750 1750 1700
 Connection ~ 1600 1750
-Wire Wire Line
-	1750 2150 1750 2100
 Connection ~ 1400 2150
 NoConn ~ 25300 21100
@@
 NoConn ~ 22700 19000
 $Comp
-L GND #PWR069
+L GND #PWR067
 U 1 1 55A8B51F
 P 25650 12700
-F 0 "#PWR069" H 25650 12450 50  0001 C CNN
+F 0 "#PWR067" H 25650 12450 50  0001 C CNN
 F 1 "GND" H 25650 12550 50  0000 C CNN
 F 2 "" H 25650 12700 60  0000 C CNN
@@
 $EndComp
 $Comp
-L +12V #PWR070
+L +12V #PWR068
 U 1 1 55A8B66F
 P 25650 11750
-F 0 "#PWR070" H 25650 11600 50  0001 C CNN
+F 0 "#PWR068" H 25650 11600 50  0001 C CNN
 F 1 "+12V" H 25650 11890 50  0000 C CNN
 F 2 "" H 25650 11750 60  0000 C CNN
@@
 	25650 12700 25650 12600
 $Comp
-L GND #PWR071
+L GND #PWR069
 U 1 1 55A948C3
 P 12150 18400
-F 0 "#PWR071" H 12150 18150 50  0001 C CNN
+F 0 "#PWR069" H 12150 18150 50  0001 C CNN
 F 1 "GND" H 12150 18250 50  0000 C CNN
 F 2 "" H 12150 18400 60  0000 C CNN
@@
 $EndComp
 $Comp
-L +12V #PWR072
+L +12V #PWR070
 U 1 1 55A94A13
 P 12200 19200
-F 0 "#PWR072" H 12200 19050 50  0001 C CNN
+F 0 "#PWR070" H 12200 19050 50  0001 C CNN
 F 1 "+12V" H 12200 19340 50  0000 C CNN
 F 2 "" H 12200 19200 60  0000 C CNN
@@
 Connection ~ 2900 2800
 $Comp
-L PWR_FLAG #FLG073
+L PWR_FLAG #FLG071
 U 1 1 55AB4E3C
 P 1150 1350
-F 0 "#FLG073" H 1150 1445 50  0001 C CNN
+F 0 "#FLG071" H 1150 1445 50  0001 C CNN
 F 1 "PWR_FLAG" H 1150 1530 50  0000 C CNN
 F 2 "" H 1150 1350 60  0000 C CNN
@@
 $EndComp
 Wire Wire Line
-	950  1400 1750 1400
-Wire Wire Line
 	1150 1400 1150 1350
 Wire Wire Line
@@
 Connection ~ 1150 1400
 $Comp
-L +6V #PWR074
+L +6V #PWR072
 U 1 1 55AB54A2
 P 1600 1300
-F 0 "#PWR074" H 1600 1150 50  0001 C CNN
+F 0 "#PWR072" H 1600 1150 50  0001 C CNN
 F 1 "+6V" H 1600 1440 50  0000 C CNN
 F 2 "" H 1600 1300 60  0000 C CNN
@@
 	1    0    0    -1
 $EndComp
+Connection ~ 1600 1400
+NoConn ~ 4350 11700
+Wire Wire Line
+	950  1400 1600 1400
 $Comp
-L VCC #PWR075
-U 1 1 55AD1FF1
-P 1750 1350
-F 0 "#PWR075" H 1750 1200 50  0001 C CNN
-F 1 "VCC" H 1750 1500 50  0000 C CNN
-F 2 "" H 1750 1350 60  0000 C CNN
-F 3 "" H 1750 1350 60  0000 C CNN
-	1    1750 1350
+L GND #PWR073
+U 1 1 55AA438D
+P 20600 3250
+F 0 "#PWR073" H 20600 3000 50  0001 C CNN
+F 1 "GND" H 20600 3100 50  0000 C CNN
+F 2 "" H 20600 3250 60  0000 C CNN
+F 3 "" H 20600 3250 60  0000 C CNN
+	1    20600 3250
 	1    0    0    -1
 $EndComp
 Wire Wire Line
-	1750 1400 1750 1350
-Connection ~ 1600 1400
-NoConn ~ 4350 11700
+	20600 3250 20600 3050
+$Comp
+L +5V #PWR074
+U 1 1 55AA47FD
+P 20600 2600
+F 0 "#PWR074" H 20600 2450 50  0001 C CNN
+F 1 "+5V" H 20600 2740 50  0000 C CNN
+F 2 "" H 20600 2600 60  0000 C CNN
+F 3 "" H 20600 2600 60  0000 C CNN
+	1    20600 2600
+	1    0    0    -1
+$EndComp
+Wire Wire Line
+	20600 2850 20600 2600
+$Comp
+L GND-RESCUE-congoBongo #PWR075
+U 1 1 55ABDA33
+P 21350 20100
+F 0 "#PWR075" H 21350 20100 30  0001 C CNN
+F 1 "GND" H 21350 20030 30  0001 C CNN
+F 2 "" H 21350 20100 60  0000 C CNN
+F 3 "" H 21350 20100 60  0000 C CNN
+	1    21350 20100
+	1    0    0    -1
+$EndComp
+$Comp
+L 74LS06 U6
+U 1 1 55ABDA39
+P 21950 19750
+F 0 "U6" H 22145 19865 60  0000 C CNN
+F 1 "7416" H 22140 19625 60  0000 C CNN
+F 2 "~" H 21950 19750 60  0000 C CNN
+F 3 "~" H 21950 19750 60  0000 C CNN
+	1    21950 19750
+	1    0    0    -1
+$EndComp
+Wire Wire Line
+	21500 19750 21350 19750
+Wire Wire Line
+	21350 19750 21350 20100
+Wire Wire Line
+	22400 19750 22700 19750
+NoConn ~ 22700 19750
+Wire Wire Line
+	950  1750 1600 1750
+Wire Wire Line
+	950  2150 1400 2150
+Connection ~ 3000 10250
+$Comp
+L GND #PWR076
+U 1 1 55B164A7
+P 3550 11900
+F 0 "#PWR076" H 3550 11650 50  0001 C CNN
+F 1 "GND" H 3550 11750 50  0000 C CNN
+F 2 "" H 3550 11900 60  0000 C CNN
+F 3 "" H 3550 11900 60  0000 C CNN
+	1    3550 11900
+	1    0    0    -1
+$EndComp
+$Comp
+L +5V #PWR077
+U 1 1 55B165FB
+P 3550 10800
+F 0 "#PWR077" H 3550 10650 50  0001 C CNN
+F 1 "+5V" H 3550 10940 50  0000 C CNN
+F 2 "" H 3550 10800 60  0000 C CNN
+F 3 "" H 3550 10800 60  0000 C CNN
+	1    3550 10800
+	1    0    0    -1
+$EndComp
+$Comp
+L +5V #PWR078
+U 1 1 55B1674F
+P 5550 11750
+F 0 "#PWR078" H 5550 11600 50  0001 C CNN
+F 1 "+5V" H 5550 11890 50  0000 C CNN
+F 2 "" H 5550 11750 60  0000 C CNN
+F 3 "" H 5550 11750 60  0000 C CNN
+	1    5550 11750
+	1    0    0    -1
+$EndComp
+$Comp
+L GND #PWR079
+U 1 1 55B168A3
+P 5500 10800
+F 0 "#PWR079" H 5500 10550 50  0001 C CNN
+F 1 "GND" H 5500 10650 50  0000 C CNN
+F 2 "" H 5500 10800 60  0000 C CNN
+F 3 "" H 5500 10800 60  0000 C CNN
+	1    5500 10800
+	1    0    0    -1
+$EndComp
+Wire Wire Line
+	3550 11900 3550 11750
+Wire Wire Line
+	3550 11050 3550 10800
+Wire Wire Line
+	5350 11000 5350 10650
+Wire Wire Line
+	5350 10650 5500 10650
+Wire Wire Line
+	5500 10650 5500 10800
+Wire Wire Line
+	5550 11750 5550 11900
+Wire Wire Line
+	5550 11900 5350 11900
+Wire Wire Line
+	5350 11900 5350 11400
+$Comp
+L C-RESCUE-congoBongo C61
+U 1 1 55B46AD5
+P 27550 20500
+F 0 "C61" H 27550 20600 40  0000 L CNN
+F 1 "1u" H 27556 20415 40  0000 L CNN
+F 2 "~" H 27588 20350 30  0000 C CNN
+F 3 "~" H 27550 20500 60  0000 C CNN
+	1    27550 20500
+	0    1    1    0
+$EndComp
+$Comp
+L R-RESCUE-congoBongo R94
+U 1 1 55B46ADB
+P 28400 20500
+F 0 "R94" V 28480 20500 40  0000 C CNN
+F 1 "51k" V 28407 20501 40  0000 C CNN
+F 2 "~" V 28330 20500 30  0000 C CNN
+F 3 "~" H 28400 20500 30  0000 C CNN
+	1    28400 20500
+	0    1    1    0
+$EndComp
+Wire Wire Line
+	27750 20500 28150 20500
 $EndSCHEMATC

Commit message: Fix C47 value from 470u to 470p
Parts:
- C47: value 470u -> 470p
- D7: value DIODE -> 1S2075
Changed lines of the file:
@@
 P 7200 3350
 F 0 "C47" H 7200 3450 40  0000 L CNN
-F 1 "470u" H 7206 3265 40  0000 L CNN
+F 1 "470p" H 7206 3265 40  0000 L CNN
 F 2 "~" H 7238 3200 30  0000 C CNN
 F 3 "~" H 7200 3350 60  0000 C CNN
@@
 P 5300 17550
 F 0 "D7" H 5300 17650 40  0000 C CNN
-F 1 "DIODE" H 5300 17450 40  0000 C CNN
+F 1 "1S2075" H 5300 17450 40  0000 C CNN
 F 2 "~" H 5300 17550 60  0000 C CNN
 F 3 "~" H 5300 17550 60  0000 C CNN
