File: kicad/congoBongo/congoBongo.sch (KiCad schematic (older format))
At the start: 144 parts, among them Q2 2SC1941{ECB}, U13 MB3614, U15 G501534, U16 MB3614, U17 MB3614, U18 4001, U19 4538, U20 MM5837, U6 7416

Commit message: Moving to kicad 5.1.5
Updated congoBongo. This will become a reference kicad schematics for conversion to netlist.
This is work in progress. Watch out for changes to README.md.
Parts:
- removed I_BASS_DRUM0, I_CONGA_H0, I_CONGA_L0, I_GORILLA0, I_RIM0, I_V0, I_V12, I_V5, I_V6: 0, symbol CONN_01X01
- removed U19: 4538, symbol 4538
- added unit 5 of U13
- added unit 5 of U16
- added unit 5 of U17
- added unit 5 of U18
- added U19: 4538, symbol 4xxx:4538
- added unit 7 of U6
- added YA_V12: 12, symbol netlist:ANALOG_INPUT
- added YA_V5: 5, symbol netlist:ANALOG_INPUT
- added YA_V6: 6, symbol netlist:ANALOG_INPUT
- added YT_BASS_DRUM0, YT_CONGA_H0, YT_CONGA_L0, YT_GORIALLA0, YT_RIM0: 0, symbol netlist:TTL_INPUT
- C20, C21, C22, C23, C24, C25, C26, C27, C28, C29, C30, C31, C32, C33, C34, C35, C36, C37, C38, C39, C40, C41, C42, C43, C44, C45, C46, C47, C48, C49, C50, C51, C52, C53, C54, C55, C56, C57, C58, C59, C60, C61, C62: symbol C-RESCUE-congoBongo -> Device:C
- D1, D2, D3, D5, D6, D7, D8: symbol DIODE -> Device:D
- D4: value DIODE -> 1S2075; symbol DIODE -> Device:D
- O_AUDIO0: symbol CONN_01X01 -> MAME:CONN_01X01
- Q2: value 2SC1941{ECB} -> 2SC1941; symbol 2SC1941 -> Device:Q_NPN_ECB; Spice_Model (none) -> 2SC1941; Spice_Netlist_Enabled (none) -> Y; Spice_Node_Sequence (none) -> 2 3 1; Spice_Primitive (none) -> Q
- R21, R22, R23, R24, R25, R26, R27, R28, R29, R30, R31, R32, R33, R34, R35, R36, R37, R38, R39, R40, R41, R42, R43, R44, R45, R46, R47, R48, R49, R50, R51, R52, R53, R54, R55, R56, R57, R58, R59, R60, R61, R62, R63, R64, R65, R66, R67, R68, R69, R70, R71, R72, R73, R74, R75, R76, R77, R78, R79, R80, R81, R82, R83, R84, R85, R86, R87, R88, R89, R90, R91, R92, R93, R94: symbol R-RESCUE-congoBongo -> Device:R
- U13, U16, U17: symbol LM324 -> Amplifier_Operational:LM324
- U15: symbol G501534 -> MAME:G501534
- U18: symbol 4001 -> 4xxx:4001
- U20: symbol MM5837 -> MAME:MM5837
- U6: symbol 74LS06 -> 74xx:74LS06
Connections:
- wire segments 375 -> 466

Commit message: Update congo bongo with new *_INPUT devices.
Parts:
- C49: value 220u -> 220p
- XBASS_DRUM0: renamed from YT_BASS_DRUM0; value 0 -> TTL_INPUT L=0; Spice_Lib_File (none) -> nlspice.lib
- XCONGA_H0: renamed from YT_CONGA_H0; value 0 -> TTL_INPUT L=0
- XCONGA_L0: renamed from YT_CONGA_L0; value 0 -> TTL_INPUT L=0; Spice_Lib_File (none) -> nlspice.lib
- XGORIALLA0: renamed from YT_GORIALLA0; value 0 -> TTL_INPUT L=0; Spice_Lib_File (none) -> nlspice.lib
- XRIM0: renamed from YT_RIM0; value 0 -> TTL_INPUT L=0; Spice_Lib_File (none) -> nlspice.lib
- XV12: renamed from YA_V12; value 12 -> ANALOG_INPUT V=12; Spice_Lib_File (none) -> nlspice.lib
- XV5: renamed from YA_V5; value 5 -> ANALOG_INPUT V=5; Spice_Lib_File (none) -> nlspice.lib
- XV6: renamed from YA_V6; value 6 -> ANALOG_INPUT V=6; Spice_Lib_File (none) -> nlspice.lib
Changed lines of the file:
@@
 P 11950 3350
 F 0 "C49" H 11950 3450 40  0000 L CNN
-F 1 "220u" H 11956 3265 40  0000 L CNN
+F 1 "220p" H 11956 3265 40  0000 L CNN
 F 2 "~" H 11988 3200 30  0000 C CNN
 F 3 "~" H 11950 3350 60  0000 C CNN
@@
 	17350 19500 17350 19700
 $Comp
-L netlist:TTL_INPUT YT_GORIALLA0
+L netlist:TTL_INPUT XGORIALLA0
 U 1 1 5E382240
 P 1250 11300
-F 0 "YT_GORIALLA0" H 1072 11346 50  0000 R CNN
-F 1 "0" H 1072 11255 50  0000 R CNN
+F 0 "XGORIALLA0" H 1072 11346 50  0000 R CNN
+F 1 "TTL_INPUT L=0" H 1072 11255 50  0000 R CNN
 F 2 "" H 1250 11300 50  0001 C CNN
 F 3 "" H 1250 11300 50  0001 C CNN
+F 4 "nlspice.lib" H 1250 11300 50  0001 C CNN "Spice_Lib_File"
 	1    1250 11300
 	1    0    0    -1
@@
 $EndComp
 $Comp
-L netlist:ANALOG_INPUT YA_V5
+L netlist:ANALOG_INPUT XV5
 U 1 1 5E58FA0C
 P 750 3700
-F 0 "YA_V5" H 833 3965 50  0000 C CNN
-F 1 "5" H 833 3874 50  0000 C CNN
+F 0 "XV5" H 833 3965 50  0000 C CNN
+F 1 "ANALOG_INPUT V=5" H 833 3874 50  0000 C CNN
 F 2 "" H 750 3700 50  0001 C CNN
 F 3 "" H 750 3700 50  0001 C CNN
+F 4 "nlspice.lib" H 750 3700 50  0001 C CNN "Spice_Lib_File"
 	1    750  3700
 	1    0    0    -1
@@
 	19350 3300 19350 3450
 $Comp
-L netlist:TTL_INPUT YT_BASS_DRUM0
+L netlist:TTL_INPUT XBASS_DRUM0
 U 1 1 5E5B5F95
 P 19350 2950
-F 0 "YT_BASS_DRUM0" H 19172 2996 50  0000 R CNN
-F 1 "0" H 19172 2905 50  0000 R CNN
+F 0 "XBASS_DRUM0" H 19172 2996 50  0000 R CNN
+F 1 "TTL_INPUT L=0" H 19172 2905 50  0000 R CNN
 F 2 "" H 19350 2950 50  0001 C CNN
 F 3 "" H 19350 2950 50  0001 C CNN
+F 4 "nlspice.lib" H 19350 2950 50  0001 C CNN "Spice_Lib_File"
 	1    19350 2950
 	1    0    0    -1
@@
 $EndComp
 $Comp
-L netlist:TTL_INPUT YT_CONGA_L0
+L netlist:TTL_INPUT XCONGA_L0
 U 1 1 5E5BD47A
 P 19350 7500
-F 0 "YT_CONGA_L0" H 19172 7546 50  0000 R CNN
-F 1 "0" H 19172 7455 50  0000 R CNN
+F 0 "XCONGA_L0" H 19172 7546 50  0000 R CNN
+F 1 "TTL_INPUT L=0" H 19172 7455 50  0000 R CNN
 F 2 "" H 19350 7500 50  0001 C CNN
 F 3 "" H 19350 7500 50  0001 C CNN
+F 4 "nlspice.lib" H 19350 7500 50  0001 C CNN "Spice_Lib_File"
 	1    19350 7500
 	1    0    0    -1
@@
 $EndComp
 $Comp
-L netlist:TTL_INPUT YT_CONGA_H0
+L netlist:TTL_INPUT XCONGA_H0
 U 1 1 5E5C258F
 P 19400 12100
-F 0 "YT_CONGA_H0" H 19222 12146 50  0000 R CNN
-F 1 "0" H 19222 12055 50  0000 R CNN
+F 0 "XCONGA_H0" H 19222 12146 50  0000 R CNN
+F 1 "TTL_INPUT L=0" H 19222 12055 50  0000 R CNN
 F 2 "" H 19400 12100 50  0001 C CNN
 F 3 "" H 19400 12100 50  0001 C CNN
@@
 $EndComp
 $Comp
-L netlist:TTL_INPUT YT_RIM0
+L netlist:TTL_INPUT XRIM0
 U 1 1 5E5CD232
 P 19450 16800
-F 0 "YT_RIM0" H 19272 16846 50  0000 R CNN
-F 1 "0" H 19272 16755 50  0000 R CNN
+F 0 "XRIM0" H 19272 16846 50  0000 R CNN
+F 1 "TTL_INPUT L=0" H 19272 16755 50  0000 R CNN
 F 2 "" H 19450 16800 50  0001 C CNN
 F 3 "" H 19450 16800 50  0001 C CNN
+F 4 "nlspice.lib" H 19450 16800 50  0001 C CNN "Spice_Lib_File"
 	1    19450 16800
 	1    0    0    -1
@@
 	19700 16800 20400 16800
 $Comp
-L netlist:ANALOG_INPUT YA_V6
+L netlist:ANALOG_INPUT XV6
 U 1 1 5E58A41C
 P 750 3200
-F 0 "YA_V6" H 833 3465 50  0000 C CNN
-F 1 "6" H 833 3374 50  0000 C CNN
+F 0 "XV6" H 833 3465 50  0000 C CNN
+F 1 "ANALOG_INPUT V=6" H 833 3374 50  0000 C CNN
 F 2 "" H 750 3200 50  0001 C CNN
 F 3 "" H 750 3200 50  0001 C CNN
+F 4 "nlspice.lib" H 750 3200 50  0001 C CNN "Spice_Lib_File"
 	1    750  3200
 	1    0    0    -1
 $EndComp
 $Comp
-L netlist:ANALOG_INPUT YA_V12
+L netlist:ANALOG_INPUT XV12
 U 1 1 5E5A30E8
 P 750 2700
-F 0 "YA_V12" H 833 2965 50  0000 C CNN
-F 1 "12" H 833 2874 50  0000 C CNN
+F 0 "XV12" H 833 2965 50  0000 C CNN
+F 1 "ANALOG_INPUT V=12" H 833 2874 50  0000 C CNN
 F 2 "" H 750 2700 50  0001 C CNN
 F 3 "" H 750 2700 50  0001 C CNN
+F 4 "nlspice.lib" H 750 2700 50  0001 C CNN "Spice_Lib_File"
 	1    750  2700
 	1    0    0    -1
