File: kicad/congoBongo/page9.sch (KiCad schematic (older format))
At the start: 26 parts, among them U2 LM324

Commit message: Moving to kicad 5.1.5
Updated congoBongo. This will become a reference kicad schematics for conversion to netlist.
This is work in progress. Watch out for changes to README.md.
Parts:
- added unit 5 of U2
- C124, C51, C53, C54, C55, C56, C57, C58, C59, C66: symbol C -> Device:C
- I_SOU: symbol CONN_01X01 -> MAME:CONN_01X01
- R77, R80, R81, R82, R83, R84, R85, R86, R87, R88, R89, R90, R91: symbol R -> Device:R
- U2: value LM324 -> MB3614; symbol LM324 -> Amplifier_Operational:LM324
- U2: symbol LM324 -> Amplifier_Operational:LM324
- VR1: symbol POT -> Device:R_POT
Connections:
- wire segments 74 -> 90
